File: elec/inflatable_led/inflatable_led.kicad_pcb (KiCad board)
At the start: 2 copper layers, 6 parts, among them U1 RP2040, U2 W25Q128JVSIQTR, X1 X322512MSB4SI

Commit message: checking schematic
Parts:
- removed BTSELCH1: TS-1187A-B-A-B, local:SW-SMD_4P-L5.1-W5.1-P3.70-LS6.5-TL-2
- added BAT1: BH-18650-A5BJ003, footprints:BAT-TH_BH-18650-A5BJ003, F.Cu at (168.0, 115.8)
- added BTBOOT0: TS-1187A-B-A-B, footprints:SW-SMD_4P-L5.1-W5.1-P3.70-LS6.5-TL-2, F.Cu at (111.9, 88.6)
- added BTRESET1: TS-1187A-B-A-B, footprints:SW-SMD_4P-L5.1-W5.1-P3.70-LS6.5-TL-2, F.Cu at (106.6, 103.9)
- added BTRESET2: TS-1187A-B-A-B, footprints:SW-SMD_4P-L5.1-W5.1-P3.70-LS6.5-TL-2, F.Cu at (133.5, 142.6)
- added C14: 10nF, Capacitor_SMD:C_0402_1005Metric, F.Cu at (124.7, 93.9)
- added C20: 100nF, Capacitor_SMD:C_0805_2012Metric, F.Cu at (167.5, 128.2)
- added C21: 100nF, Capacitor_SMD:C_0805_2012Metric, F.Cu at (176.1, 134.8)
- added C22: 10nF, Capacitor_SMD:C_0402_1005Metric, F.Cu at (166.7, 143.2)
- added D1: MBR0540T1G, footprints:SOD-123_L2.8-W1.8-LS3.7-RD, F.Cu at (154.4, 128.2)
- added D8: MBR0540T1G, footprints:SOD-123_L2.8-W1.8-LS3.7-RD, F.Cu at (154.4, 131.1)
- added D9: MBR0540T1G, footprints:SOD-123_L2.8-W1.8-LS3.7-RD, F.Cu at (154.4, 134.0)
- added L1: 1255AY-100M=P3, footprints:IND-SMD_L6.0-W6.0, F.Cu at (161.1, 130.5)
- added LED1: KT-0603R, footprints:LED0603-RD, F.Cu at (159.1, 135.6)
- added LED2: KT-0603R, footprints:LED0603-RD, F.Cu at (159.1, 138.2)
- added R10: 5.1K, Resistor_SMD:R_0402_1005Metric, F.Cu at (230.9, 78.1)
- added R11: 5.1K, Resistor_SMD:R_0402_1005Metric, F.Cu at (230.9, 75.2)
- added R12: 100R, Resistor_SMD:R_0402_1005Metric, F.Cu at (139.6, 131.7)
- added R13: 10K, Resistor_SMD:R_0402_1005Metric, F.Cu at (114.2, 131.4)
- added R14: 10K, Resistor_SMD:R_0402_1005Metric, F.Cu at (114.2, 134.3)
- added R15: 10K, Resistor_SMD:R_0402_1005Metric, F.Cu at (139.6, 137.7)
- added R5: 10K, Resistor_SMD:R_0402_1005Metric, F.Cu at (97.6, 80.4)
- added R7: 600R, Resistor_SMD:R_0402_1005Metric, F.Cu at (139.6, 129.7)
- added TPCC1: TestPoint, TestPoint:TestPoint_Pad_D1.5mm, F.Cu at (223.2, 78.1)
- added TPCC2: TestPoint, TestPoint:TestPoint_Pad_D1.5mm, F.Cu at (222.9, 74.5)
- added U3: TPS61165DRVR, footprints:WSON-6_L2.0-W2.0-P0.65-TL-EP, F.Cu at (167.5, 138.6)
- added U4: BQ24040DSQR, footprints:WSON-10_L2.0-W2.0-P0.40-BL-EP, F.Cu at (196.8, 95.5)
- added U5: AMS1117-3.3, footprints:SOT-223-3_L6.5-W3.4-P2.30-LS7.0-BR, F.Cu at (145.7, 139.9)
- added U6: F.0603.00026/P2-0603B1TS2-06T-001, footprints:LED0603-RD, F.Cu at (159.1, 140.9)
- added U7: SI2323DS, footprints:SOT-23-3_L2.9-W1.3-P1.90-LS2.4-BR, F.Cu at (167.4, 134.9)
- added USB2: KH-TYPE-C-16P, footprints:USB-C-SMD_KH-TYPE-C-16P, F.Cu at (236.7, 76.9)
- moved C13 35.4 mm to (109.8, 71.7)
- moved U1 35.4 mm to (135.7, 74.2)
- moved X1 35.4 mm to (133.8, 81.1)
- moved R4 35.4 mm to (107.0, 71.7)
- moved U2 35.4 mm to (127.7, 74.8)
Connections:
- C13 pad 1: Net-(BTSELCH1-A) -> /run
- R4 pad 2: Net-(BTSELCH1-A) -> /run
- U1 pad 19: unconnected-(U1-TESTEN-Pad19) -> GND
- U1 pad 26: unconnected-(U1-RUN-Pad26) -> /run
- U1 pad 38: unconnected-(U1-GPIO26_ADC0-Pad38) -> /BAT_SENSE
- U1 pad 43: unconnected-(U1-ADC_AVDD-Pad43) -> +3V3
- U1 pad 5: unconnected-(U1-GPIO3-Pad5) -> /LED_ON
- U1 pad 6: unconnected-(U1-GPIO4-Pad6) -> /DIM_CTRL

Commit message: layout almost done + CI
Parts:
- removed BTRESET2: TS-1187A-B-A-B, footprints:SW-SMD_4P-L5.1-W5.1-P3.70-LS6.5-TL-2
- removed LED1, LED2: KT-0603R, footprints:LED0603-RD
- added BAT2: BH-18650-A5BJ003, footprints:BAT-TH_BH-18650-A5BJ003, F.Cu at (101.4, 112.2)
- added C1: 20pF, Capacitor_SMD:C_0402_1005Metric, F.Cu at (88.2, 58.4)
- added C10: 100nF, Capacitor_SMD:C_0402_1005Metric, F.Cu at (103.6, 62.8)
- added C11: 100nF, Capacitor_SMD:C_0402_1005Metric, F.Cu at (90.7, 64.4)
- added C12: 1uF, Capacitor_SMD:C_0805_2012Metric, F.Cu at (107.1, 65.3)
- added C15: 220nF, Capacitor_SMD:C_0603_1608Metric, F.Cu at (77.8, 129.2)
- added C16: 4.7uF, Capacitor_SMD:C_0805_2012Metric, F.Cu at (81.2, 125.0)
- added C17: 1uF, Capacitor_SMD:C_0805_2012Metric, F.Cu at (81.3, 134.9)
- added C18: 1uF, Capacitor_SMD:C_0805_2012Metric, F.Cu at (123.1, 126.1)
- added C19: 1uF, Capacitor_SMD:C_0805_2012Metric, F.Cu at (123.1, 129.8)
- added C2: 20pF, Capacitor_SMD:C_0402_1005Metric, F.Cu at (90.8, 61.4)
- added C3: 100nF, Capacitor_SMD:C_0402_1005Metric, F.Cu at (100.8, 68.5)
- added C4: 100nF, Capacitor_SMD:C_0402_1005Metric, F.Cu at (103.6, 67.3)
- added C5: 100nF, Capacitor_SMD:C_0402_1005Metric, F.Cu at (102.3, 58.8)
- added C6: 100nF, Capacitor_SMD:C_0402_1005Metric, F.Cu at (91.2, 63.3)
- added C7: 100nF, Capacitor_SMD:C_0402_1005Metric, F.Cu at (96.5, 68.6)
- added C8: 1uF, Capacitor_SMD:C_0805_2012Metric, F.Cu at (103.6, 69.6)
- added C9: 100nF, Capacitor_SMD:C_0402_1005Metric, F.Cu at (103.6, 66.2)
- added D10: LED, footprints:GW JTLPS1EM, B.Cu at (80.0, 80.0)
- added D11: LED, footprints:GW JTLPS1EM, B.Cu at (100.0, 80.0)
- added D12: LED, footprints:GW JTLPS1EM, B.Cu at (120.0, 80.0)
- added D13: LED, footprints:GW JTLPS1EM, B.Cu at (120.0, 120.0)
- added D14: LED, footprints:GW JTLPS1EM, B.Cu at (100.0, 120.0)
- added D15: LED, footprints:GW JTLPS1EM, B.Cu at (80.0, 120.0)
- added D2: LED, footprints:GW JTLPS1EM, F.Cu at (93.9, 144.3)
- added D3: LED, footprints:GW JTLPS1EM, F.Cu at (102.8, 144.3)
- added D4: LED, footprints:GW JTLPS1EM, F.Cu at (144.0, 116.1)
- added D5: LED, footprints:GW JTLPS1EM, F.Cu at (103.8, 52.7)
- added D6: LED, footprints:GW JTLPS1EM, F.Cu at (96.5, 52.7)
- added D7: LED, footprints:GW JTLPS1EM, F.Cu at (57.4, 84.4)
- added H1: MountingHole, MountingHole:MountingHole_3.2mm_M3_Pad_Via, F.Cu at (75.0, 60.8)
- added H2: MountingHole, MountingHole:MountingHole_3.2mm_M3_Pad_Via, F.Cu at (75.0, 139.2)
- added H3: MountingHole, MountingHole:MountingHole_3.2mm_M3_Pad_Via, F.Cu at (125.0, 60.8)
- added H4: MountingHole, MountingHole:MountingHole_3.2mm_M3_Pad_Via, F.Cu at (125.0, 139.2)
- added J1: Header-Male-2.54_1x20, footprints:HDR-TH_20P-P2.54-V-M-1, F.Cu at (101.4, 100.0)
- added J2: Conn_01x02_Pin, Connector_PinHeader_2.54mm:PinHeader_1x02_P2.54mm_Vertical, F.Cu at (68.1, 128.3)
- added J3: Conn_01x02_Pin, Connector_PinHeader_2.54mm:PinHeader_1x02_P2.54mm_Vertical, F.Cu at (115.1, 128.7)
- added LED_CHG_2: KT-0603R, footprints:LED0603-RD, F.Cu at (120.4, 131.2)
- added LED_PG_1: KT-0603R, footprints:LED0603-RD, F.Cu at (120.3, 124.9)
- added R1: 1k, Resistor_SMD:R_0402_1005Metric, F.Cu at (88.3, 64.5)
- added R16: 100R, Resistor_SMD:R_0402_1005Metric, F.Cu at (97.1, 129.9)
- added R2: 27R, Resistor_SMD:R_0402_1005Metric, F.Cu at (103.6, 63.8)
- added R3: 27R, Resistor_SMD:R_0402_1005Metric, F.Cu at (103.6, 64.8)
- added R6: 0.8R, Resistor_SMD:R_0805_2012Metric_Pad1.20x1.40mm_HandSolder, F.Cu at (72.1, 128.2)
- added R8: 100R, Resistor_SMD:R_0402_1005Metric, F.Cu at (125.9, 126.5)
- added R9: 100R, Resistor_SMD:R_0402_1005Metric, F.Cu at (125.9, 129.5)
- added SW1: TS-1093C-A7B2-D1, footprints:SW-TH_TS-1093C-A7B3-D1, F.Cu at (58.6, 100.0)
- added TP3: TestPoint, TestPoint:TestPoint_Pad_D1.5mm, F.Cu at (129.2, 75.0)
- added TP4: TestPoint, TestPoint:TestPoint_Pad_D1.5mm, F.Cu at (89.9, 66.2)
- added TP5: TestPoint, TestPoint:TestPoint_Pad_D1.5mm, F.Cu at (87.3, 66.3)
- added TP6: TestPoint, TestPoint:TestPoint_Pad_D1.5mm, F.Cu at (128.9, 127.5)
- added TP_DIM_CTRL_1: TestPoint, TestPoint:TestPoint_Pad_D1.5mm, F.Cu at (84.9, 124.1)
- added TP_LED_ON1: TestPoint, TestPoint:TestPoint_Pad_D1.5mm, F.Cu at (96.9, 133.7)
- added TP_POWER_OR_1: TestPoint, TestPoint:TestPoint_Pad_D1.5mm, F.Cu at (134.5, 128.6)
- added TP_SW_LED1: TestPoint, TestPoint:TestPoint_Pad_D1.5mm, F.Cu at (93.0, 126.7)
- moved C22 118.4 mm to (59.5, 92.8)
- moved R15 94.0 mm to (57.0, 92.8)
- moved USB2 93.9 mm to (145.6, 100.0)
- moved R10 91.3 mm to (144.7, 108.3), turned to -90 degrees
- moved R11 88.0 mm to (144.6, 92.3), turned to 90 degrees
- moved U3 86.8 mm to (81.2, 129.2)
- moved TPCC1 86.4 mm to (142.2, 108.3)
- moved U4 83.0 mm to (120.4, 128.1), turned to 180 degrees
- moved TPCC2 82.5 mm to (142.4, 92.4)
- moved C21 74.8 mm to (101.5, 128.3), turned to -90 degrees
- moved U7 73.5 mm to (94.0, 130.1)
- moved D1 73.2 mm to (81.3, 132.4)
- moved L1 73.1 mm to (88.0, 129.2), turned to -90 degrees
- moved BAT1 72.2 mm to (101.4, 87.9)
- moved R14 61.8 mm to (131.5, 75.0), turned to 0 degrees
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Connections:
- BTBOOT0 pad 1: /qspi_ss -> /QSPI_SS
- BTBOOT0 pad 2: /qspi_ss -> /QSPI_SS
- C14 pad 1: /qspi_ss -> /QSPI_SS
- C20 pad 1: VBUS -> /POWER_IN_OR
- R5 pad 2: /qspi_ss -> /QSPI_SS
- U1 pad 1: +3V3 -> +3.3V
- U1 pad 10: +3V3 -> +3.3V
- U1 pad 12: unconnected-(U1-GPIO9-Pad12) -> Net-(U1-GPIO9)
- U1 pad 13: unconnected-(U1-GPIO10-Pad13) -> Net-(U1-GPIO10)
- U1 pad 14: unconnected-(U1-GPIO11-Pad14) -> Net-(U1-GPIO11)
- U1 pad 15: unconnected-(U1-GPIO12-Pad15) -> Net-(U1-GPIO12)
- U1 pad 16: unconnected-(U1-GPIO13-Pad16) -> Net-(U1-GPIO13)
- U1 pad 17: unconnected-(U1-GPIO14-Pad17) -> Net-(U1-GPIO14)
- U1 pad 18: unconnected-(U1-GPIO15-Pad18) -> Net-(U1-GPIO15)
- U1 pad 22: +3V3 -> +3.3V
- U1 pad 24: unconnected-(U1-SWCLK-Pad24) -> /SWCLK
- U1 pad 25: unconnected-(U1-SWD-Pad25) -> /SWD
- U1 pad 27: unconnected-(U1-GPIO16-Pad27) -> Net-(U1-GPIO16)
- U1 pad 28: unconnected-(U1-GPIO17-Pad28) -> Net-(U1-GPIO17)
- U1 pad 29: unconnected-(U1-GPIO18-Pad29) -> Net-(U1-GPIO18)
- U1 pad 30: unconnected-(U1-GPIO19-Pad30) -> Net-(U1-GPIO19)
- U1 pad 31: unconnected-(U1-GPIO20-Pad31) -> Net-(U1-GPIO20)
- U1 pad 32: unconnected-(U1-GPIO21-Pad32) -> Net-(U1-GPIO21)
- U1 pad 33: +3V3 -> +3.3V
- U1 pad 34: unconnected-(U1-GPIO22-Pad34) -> Net-(U1-GPIO22)
- U1 pad 35: unconnected-(U1-GPIO23-Pad35) -> Net-(U1-GPIO23)
- U1 pad 36: unconnected-(U1-GPIO24-Pad36) -> Net-(U1-GPIO24)
- U1 pad 37: unconnected-(U1-GPIO25-Pad37) -> Net-(U1-GPIO25)
- U1 pad 38: /BAT_SENSE -> Net-(U1-GPIO26_ADC0)
- U1 pad 39: unconnected-(U1-GPIO27_ADC1-Pad39) -> Net-(U1-GPIO27_ADC1)
- U1 pad 40: unconnected-(U1-GPIO28_ADC2-Pad40) -> Net-(U1-GPIO28_ADC2)
- U1 pad 41: unconnected-(U1-GPIO29_ADC3-Pad41) -> /BAT_SENSE
- U1 pad 42: +3V3 -> +3.3V
- U1 pad 43: +3V3 -> +3.3V
- U1 pad 44: unconnected-(U1-VREG_IN-Pad44) -> +3.3V
- U1 pad 45: unconnected-(U1-VREG_VOUT-Pad45) -> +1V0
- U1 pad 48: unconnected-(U1-USB_VDD-Pad48) -> +3.3V
- U1 pad 49: +3V3 -> +3.3V
- U1 pad 7: unconnected-(U1-GPIO5-Pad7) -> /ON_OFF_BT
- U7 pad 1: /LED_ON -> Net-(U7-G)
Routing:
- net +3.3V: track 0.00 -> 222.1 mm, vias 0 -> 7
- net /LED_ON: track 0.00 -> 113.8 mm, vias 0 -> 2
- net /DIM_CTRL: track 0.00 -> 112.7 mm, vias 0 -> 4
- net +BATT: track 0.00 -> 110.7 mm, vias 0 -> 2
- net /LED_SOURCE: track 0.00 -> 85.9 mm
- net Net-(D4-K): track 0.00 -> 82.1 mm
- net /ON_OFF_BT: track 0.00 -> 74.7 mm, vias 0 -> 1
- net /LED_SINK: track 0.00 -> 72.5 mm
- net VBUS: track 0.00 -> 63.3 mm, vias 0 -> 4
- net /USB_DP: track 0.00 -> 61.8 mm, vias 0 -> 2
- net /USB_DM: track 0.00 -> 61.2 mm, vias 0 -> 4
- net Net-(U1-GPIO9): track 0.00 -> 60.3 mm
- net Net-(U1-GPIO10): track 0.00 -> 58.1 mm
- net Net-(U1-GPIO11): track 0.00 -> 55.5 mm
- net Net-(U1-GPIO15): track 0.00 -> 55.2 mm
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- added copper zone on B.Cu, net GND
- added copper zone on F.Cu, net GND
Other:
- board outline added: 100.1 x 100 mm

Commit message: fix all unconnected items
Parts:
- moved R14 0.65 mm to (131.1, 75.5), turned to -90 degrees
- moved LED_PG_1 0.22 mm to (120.2, 124.7)
Routing:
- net GND: track 3.97 -> 18.1 mm, vias 107 -> 132
- net Net-(U4-ISET): track 3.86 -> 4.91 mm
