File: elec/inflatable_led/inflatable_led.kicad_pcb (KiCad board)
At the start: 4 copper layers, 91.8 x 92 mm, 103 parts, among them CN1 S2B-PH-SM4-TB(LF)(SN), J1 Conn_01x10, J2 Conn_01x02_Pin, J3 Conn_01x02_Pin, J4 USB4205-GF-A_REVA, Q1 2N7002KW_R1_00001, U1 RP2040, U2 W25Q128JVSIQTR, U3 TPS61165DRVR, U4 BQ25601DRTWR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

Commit message: add a few silkscreen items
Other:
- outline, holes or cut-outs redrawn
- board text added: "Charge"
- board text added: "Inflatable led lamp V2 Zurich, Oct. 2024"
- board text added: "Power good"
Changed lines of the file:
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@@
 			(layer "F.SilkS"
 				(type "Top Silk Screen")
+				(color "Black")
 			)
 			(layer "F.Paste"
@@
 			(layer "B.SilkS"
 				(type "Bottom Silk Screen")
+				(color "Black")
 			)
 			(copper_finish "None")
@@
 		(net 57)
 	)
+	(gr_line
+		(start 128.37 123.8)
+		(end 117.87 123.8)
+		(stroke
+			(width 0.1)
+			(type default)
+		)
+		(layer "F.SilkS")
+	)
 	(gr_circle
 		(center 101.369979 129.999989)
@@
 		(layer "Edge.Cuts")
 	)
-	(gr_circle
-		(center 101.369979 99.999989)
-		(end 101.369979 99.949989)
-		(stroke
-			(width 0.1)
-			(type default)
-		)
-		(fill none)
-		(layer "Edge.Cuts")
-	)
 	(gr_arc
 		(start 119.556513 137.49999)
@@
 		(layer "Edge.Cuts")
 	)
+	(gr_text "Inflatable led lamp V2\nZurich, Oct. 2024"
+		(at 108.57 101.45 -0)
+		(layer "B.SilkS")
+		(effects
+			(font
+				(size 1 1)
+				(thickness 0.1)
+			)
+			(justify left bottom mirror)
+		)
+	)
+	(gr_text "Charge"
+		(at 123.42 123.25 0)
+		(layer "F.SilkS")
+		(effects
+			(font
+				(size 1 1)
+				(thickness 0.1)
+			)
+			(justify left bottom)
+		)
+	)
 	(gr_text "Reset"
 		(at 92.77 64.4 0)
@@
 		)
 	)
+	(gr_text "Power\ngood"
+		(at 123.72 126.8 0)
+		(layer "F.SilkS")
+		(effects
+			(font
+				(size 1 1)
+				(thickness 0.1)
+			)
+			(justify left bottom)
+		)
+	)
 	(segment
 		(start 91.9 74.32)
@@
 	)
 	(via
-		(at 101.52 98.7)
+		(at 101.67 96.15)
 		(size 0.6)
 		(drill 0.3)
@@
 			"b96a1250-9c43-4645-9d3f-9ffb085f25db" "d066847d-41f8-4345-83ce-473f2e9587f0"
 			"e8af5358-4585-49f8-a4d1-87bf1bf25563" "e9222337-db0b-4d58-852e-06fcdafc1991"
-			"e926688b-d46e-47e4-b74a-13ca6cd19f59" "ef7103cd-dc1f-435d-a2b8-10566d60633a"
-			"f09b3a5a-daed-45cd-9ede-f8b5fe0e59a2" "f1337bdd-6786-4137-9905-23ae5957696e"
+			"e926688b-d46e-47e4-b74a-13ca6cd19f59" "f09b3a5a-daed-45cd-9ede-f8b5fe0e59a2"
+			"f1337bdd-6786-4137-9905-23ae5957696e"
 		)
 	)

Commit message: add OR gate to circuit
Parts:
- added TP10: TestPoint, TestPoint:TestPoint_Pad_D1.0mm, F.Cu at (111.0, 75.5)
- added TP9: TestPoint, TestPoint:TestPoint_Pad_D1.0mm, F.Cu at (114.5, 70.0)
- added U9: 74LVC1G32SE-7, footprints:SOT-353_L2.0-W1.2-P0.65-LS2.1-BL, F.Cu at (114.3, 76.1)
- R16: value 100R -> 100
- R18: value 10K -> 1k
Connections:
- J1 pad 6: /PWR_EN -> /LDO_EN
- U8 pad 3: /PWR_EN -> /LDO_EN
Routing:
- net /LDO_EN: track 0.00 -> 67.1 mm, vias 0 -> 2
- net /PWR_EN: track 75.2 -> 8.10 mm, vias 2 -> 0
- net VCC: track 90.6 -> 93.2 mm
- net GND: track 45.5 -> 46.7 mm, vias 68 -> 69
- net VBUS: track 15.3 -> 16.4 mm, vias 11 -> 13
